Commit message: delete push

File: model/manipulator.urdf (robot description, URDF)
Before this commit: robot manipulator, 6 links, 5 joints
Links:
- link base_link: geometry collision mesh filename=/home/erm/rl-project/meshes/base_link.STL; visual mesh filename=/home/erm/rl-project/meshes/base_link.STL
- link link_1: geometry collision mesh filename=/home/erm/rl-project/meshes/link_1.STL; visual mesh filename=/home/erm/rl-project/meshes/link_1.STL
- link link_2: geometry collision mesh filename=/home/erm/rl-project/meshes/link_2.STL; visual mesh filename=/home/erm/rl-project/meshes/link_2.STL
- link link_3: geometry collision mesh filename=/home/erm/rl-project/meshes/link_3.STL; visual mesh filename=/home/erm/rl-project/meshes/link_3.STL

Commit message: change mesh dir

File: model/manipulator.urdf (robot description, URDF)
Before this commit: robot manipulator, 6 links, 5 joints
Links:
- link base_link: geometry collision mesh filename=./meshes/base_link.STL; visual mesh filename=./meshes/base_link.STL
- link link_1: geometry collision mesh filename=./meshes/link_1.STL; visual mesh filename=./meshes/link_1.STL
- link link_2: geometry collision mesh filename=./meshes/link_2.STL; visual mesh filename=./meshes/link_2.STL
- link link_3: geometry collision mesh filename=./meshes/link_3.STL; visual mesh filename=./meshes/link_3.STL
